Commit message: robocup2024 pre-competition commits

File: mir_robots/mir_hardware_config/youbot-brsu-2/urdf/robot.urdf.xacro (robot description, xacro)
@@ -35,5 +35,6 @@
   <!-- Arm Plate moving arm 8cm foward and 45 degree rotation -->
   <xacro:full_platform name="full_platform" parent="base_link" arm_angle="${-M_PI / 4}">
-    <origin xyz="0.0 0.0 ${0.021 + 0.025 + 0.025}" rpy="0 0 0" />    <!-- ${alignment with base top + spacer height + spacer height } -->
+    <!-- <origin xyz="0.0 0.0 ${0.021 + 0.025 + 0.025}" rpy="0 0 0" />    ${alignment with base top + spacer height + spacer height } -->
+    <origin xyz="0.0 0.0 ${0.021 + 0.025 + 0.025 - 0.030}" rpy="0 0 0" />
   </xacro:full_platform>
   <xacro:youbot_arm name="arm" parent="full_platform_arm_root_link">
@@ -55,5 +56,6 @@
      <!-- camera calibration -->
       <!-- <origin xyz="0.035 0.020 0.0" rpy="0.0 1.22 0.0" /> -->
-      <origin xyz="-0.026 0.005 0.0" rpy="0.0 1.22 0.0" />
+      <!-- <origin xyz="-0.026 0.005 0.0" rpy="0.0 1.22 0.0" />   -->
+      <origin xyz="-0.034 0.008 -0.004" rpy="0.0 1.22 0.0" />
   </xacro:sensor_d435>
   <!-- tower middle camera -->

Commit message: robocup2024 changes

File: mir_robots/mir_hardware_config/youbot-brsu-2/urdf/robot.urdf.xacro (robot description, xacro)
@@ -57,5 +57,6 @@
       <!-- <origin xyz="0.035 0.020 0.0" rpy="0.0 1.22 0.0" /> -->
       <!-- <origin xyz="-0.026 0.005 0.0" rpy="0.0 1.22 0.0" />   -->
-      <origin xyz="-0.034 0.008 -0.004" rpy="0.0 1.22 0.0" />
+      <!-- <origin xyz="-0.034 0.008 -0.004" rpy="0.0 1.22 0.0" />   -->
+      <origin xyz="-0.055 0.020 0.016" rpy="0.0 1.22 0.0" />
   </xacro:sensor_d435>
   <!-- tower middle camera -->

Commit message: GO25 Pre Commit

File: mir_robots/mir_hardware_config/youbot-brsu-2/urdf/robot.urdf.xacro (robot description, xacro)
@@ -58,5 +58,6 @@
       <!-- <origin xyz="-0.026 0.005 0.0" rpy="0.0 1.22 0.0" />   -->
       <!-- <origin xyz="-0.034 0.008 -0.004" rpy="0.0 1.22 0.0" />   -->
-      <origin xyz="-0.055 0.020 0.016" rpy="0.0 1.22 0.0" />
+      <!-- <origin xyz="-0.055 0.020 0.016" rpy="0.0 1.22 0.0" />   -->
+      <origin xyz="-0.040 0.020 0.016" rpy="0.0 1.22 0.0" />
   </xacro:sensor_d435>
   <!-- tower middle camera -->

Commit message: GO25 after competition

File: mir_robots/mir_hardware_config/youbot-brsu-2/urdf/robot.urdf.xacro (robot description, xacro)
@@ -59,5 +59,6 @@
       <!-- <origin xyz="-0.034 0.008 -0.004" rpy="0.0 1.22 0.0" />   -->
       <!-- <origin xyz="-0.055 0.020 0.016" rpy="0.0 1.22 0.0" />   -->
-      <origin xyz="-0.040 0.020 0.016" rpy="0.0 1.22 0.0" />
+      <!-- <origin xyz="-0.040 0.020 0.016" rpy="0.0 1.22 0.0" />  --> <!--Pre-GermanOpen25-->
+      <origin xyz="-0.00 0.020 0.016" rpy="0.0 1.22 0.0" />
   </xacro:sensor_d435>
   <!-- tower middle camera -->

Commit message: robocup 2025 pre-commits

File: mir_robots/mir_hardware_config/youbot-brsu-2/urdf/robot.urdf.xacro (robot description, xacro)
@@ -60,5 +60,5 @@
       <!-- <origin xyz="-0.055 0.020 0.016" rpy="0.0 1.22 0.0" />   -->
       <!-- <origin xyz="-0.040 0.020 0.016" rpy="0.0 1.22 0.0" />  --> <!--Pre-GermanOpen25-->
-      <origin xyz="-0.00 0.020 0.016" rpy="0.0 1.22 0.0" />
+      <origin xyz="-0.025 0.023 0.025" rpy="0.0 1.22 0.0" />   <!--z=0.016 prev-->
   </xacro:sensor_d435>
   <!-- tower middle camera -->
@@ -116,5 +116,5 @@
     <visual>
       <geometry>
-        <box size="0.030 0.030 0.608"/>
+        <box size="0.030 0.030 0.56"/>  <!--0.608 -->
       </geometry>
       <material name="">

Commit message: updated camera pose based on calibration in Brazil

File: mir_robots/mir_hardware_config/youbot-brsu-2/urdf/robot.urdf.xacro (robot description, xacro)
@@ -55,10 +55,6 @@
   <xacro:sensor_d435 name="tower_cam3d_front_camera" parent="tower_camera_front_bolt_link" use_nominal_extrinsics="true">
      <!-- camera calibration -->
-      <!-- <origin xyz="0.035 0.020 0.0" rpy="0.0 1.22 0.0" /> -->
-      <!-- <origin xyz="-0.026 0.005 0.0" rpy="0.0 1.22 0.0" />   -->
-      <!-- <origin xyz="-0.034 0.008 -0.004" rpy="0.0 1.22 0.0" />   -->
-      <!-- <origin xyz="-0.055 0.020 0.016" rpy="0.0 1.22 0.0" />   -->
       <!-- <origin xyz="-0.040 0.020 0.016" rpy="0.0 1.22 0.0" />  --> <!--Pre-GermanOpen25-->
-      <origin xyz="-0.025 0.023 0.025" rpy="0.0 1.22 0.0" />   <!--z=0.016 prev-->
+      <origin xyz="-0.033 0.023 0.030" rpy="0.0 1.22 0.0" />
   </xacro:sensor_d435>
   <!-- tower middle camera -->
